File: hardware/Water-level-esp8266-esphome-solar-charing.kicad_pcb (KiCad board)
At the start: 2 copper layers, 60 x 60 mm, 69 parts, among them J1 RESET, J2 FLASH, J3 TTL, J4 HCR, J5 BATTERY, J6 SOLAR PANEL, Q1 AOD4184, Q2 FS8205A, U1 ESP-12E, U2 AMS1117-3.3, U3 MT3608, U4 INA219AxD, U5 CN3791, U6 DW01A

Commit message: Add files via upload
Parts:
- removed R17: 56K, Resistor_SMD:R_0805_2012Metric_Pad1.20x1.40mm_HandSolder
- J4: value HCR -> Hcr
- R13: value 100K -> 68K
- R14: value 43K -> 39K
- R15: value 22K -> 33K
- renumbered 18V3 to 12V3, 9V1 to 6V1, 12V2 to 9V2
Changed lines of the file:
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@@
 		(descr "SMD Solder Jumper, 1x1.5mm, rounded Pads, 0.3mm gap, open")
 		(tags "solder jumper open")
-		(property "Reference" "12V2"
+		(property "Reference" "9V2"
 			(at -0.035 -1.755 0)
 			(layer "F.SilkS")
@@
 			(size 1 0.5)
 			(layers "F.Cu" "F.Mask")
-			(net "Net-(12V2-B)")
+			(net "Net-(9V2-B)")
 			(pinfunction "B_2")
 			(pintype "passive")
@@
 			)
 		)
-		(property "Value" "100K"
-			(at 3.37 -0.07 0)
+		(property "Value" "68K"
+			(at 3.223 -0.07 0)
 			(layer "F.SilkS")
 			(effects
@@
 			(layers "F.Cu" "F.Mask" "F.Paste")
 			(roundrect_rratio 0.208333)
-			(net "Net-(9V1-A)")
+			(net "Net-(6V1-A)")
 			(pintype "passive")
 		)
@@
 		)
 	)
-	(footprint "Resistor_SMD:R_0805_2012Metric_Pad1.20x1.40mm_HandSolder"
-		(layer "F.Cu")
-		(at 157.88 118.93 90)
-		(descr "Resistor SMD 0805 (2012 Metric), square (rectangular) end terminal, IPC-7351 nominal with elongated pad for handsoldering. (Body size source: IPC-SM-782 page 72, https://www.pcb-3d.com/wordpress/wp-content/uploads/ipc-sm-782a_amendment_1_and_2.pdf)")
-		(tags "resistor handsolder")
-		(property "Reference" "R17"
-			(at -1.34 2.38 180)
-			(layer "F.SilkS")
-			(effects
-				(font
-					(size 0.8 0.8)
-					(thickness 0.1)
-				)
-			)
-		)
-		(property "Value" "56K"
-			(at 0.02 2.35 180)
-			(layer "F.SilkS")
-			(effects
-				(font
-					(size 0.8 0.8)
-					(thickness 0.1)
-				)
-			)
-		)
-		(property "Datasheet" ""
-			(at 0 0 90)
-			(layer "F.Fab")
-			(hide yes)
-			(effects
-				(font
-					(size 1.27 1.27)
-				)
-			)
-		)
-		(property "Description" "Resistor"
-			(at 0 0 90)
-			(layer "F.Fab")
-			(hide yes)
-			(effects
-				(font
-					(size 1.27 1.27)
-				)
-			)
-		)
-		(property "KiLib_Generator" "SMD_2terminal_chip_molded"
-			(at 0 0 90)
-			(layer "F.SilkS")
-			(hide yes)
-			(effects
-				(font
-					(size 1 1)
-					(thickness 0.15)
-				)
-			)
-		)
-		(property ki_fp_filters "R_*")
-		(sheetname "/")
-		(sheetfile "Water-level-esp8266-esphome-solar-charing.kicad_sch")
-		(units
-			(unit
-				(name "A")
-				(pins "1" "2")
-			)
-		)
-		(attr smd)
-		(duplicate_pad_numbers_are_jumpers no)
-		(fp_line
-			(start -0.227064 -0.735)
-			(end 0.227064 -0.735)
-			(stroke
-				(width 0.12)
-				(type solid)
-			)
-			(layer "F.SilkS")
-		)
-		(fp_line
-			(start -0.227064 0.735)
-			(end 0.227064 0.735)
-			(stroke
-				(width 0.12)
-				(type solid)
-			)
-			(layer "F.SilkS")
-		)
-		(fp_rect
-			(start -1.85 -0.95)
-			(end 1.85 0.95)
-			(stroke
-				(width 0.05)
-				(type solid)
-			)
-			(fill no)
-			(layer "F.CrtYd")
-		)
-		(fp_rect
-			(start -1 -0.625)
-			(end 1 0.625)
-			(stroke
-				(width 0.1)
-				(type solid)
-			)
-			(fill no)
-			(layer "F.Fab")
-		)
-		(pad "1" smd roundrect
-			(at -1 0 90)
-			(size 1.2 1.4)
-			(layers "F.Cu" "F.Mask" "F.Paste")
-			(roundrect_rratio 0.208333)
-			(net "/MPPT")
-			(pintype "passive")
-		)
-		(pad "2" smd roundrect
-			(at 1 0 90)
-			(size 1.2 1.4)
-			(layers "F.Cu" "F.Mask" "F.Paste")
-			(roundrect_rratio 0.208333)
-			(net "GND")
-			(pintype "passive")
-		)
-		(embedded_fonts no)
-		(model "${KICAD10_3DMODEL_DIR}/Resistor_SMD.3dshapes/R_0805_2012Metric.step"
-			(offset
-				(xyz 0 0 0)
-			)
-			(scale
-				(xyz 1 1 1)
-			)
-			(rotate
-				(xyz 0 0 0)
-			)
-		)
-	)
 	(footprint "Capacitor_SMD:C_1206_3216Metric_Pad1.33x1.80mm_HandSolder"
 		(layer "F.Cu")
@@
 		(descr "SMD Solder Jumper, 1x1.5mm, rounded Pads, 0.3mm gap, open")
 		(tags "solder jumper open")
-		(property "Reference" "9V1"
+		(property "Reference" "6V1"
 			(at 0.075 1.735 0)
 			(layer "F.SilkS")
@@
 			(size 1 0.5)
 			(layers "F.Cu" "F.Mask")
-			(net "Net-(9V1-A)")
+			(net "Net-(6V1-A)")
 			(pinfunction "A_1")
 			(pintype "passive")
@@
 			)
 		)
-		(property "Value" "43K"
-			(at -2.84 0.03 0)
+		(property "Value" "39K"
+			(at -3.183 0.03 0)
 			(layer "F.SilkS")
 			(effects
@@
 			(layers "F.Cu" "F.Mask" "F.Paste")
 			(roundrect_rratio 0.208333)
-			(net "Net-(12V2-B)")
+			(net "Net-(9V2-B)")
 			(pintype "passive")
 		)
@@
 		)
 		(property "Value" "200K"
-			(at -2.41 -0.58 0)
+			(at -0.165 -1.91 270)
 			(layer "F.SilkS")
 			(effects
@@
 			(at 0 -2.85 0)
 			(layer "F.SilkS")
+			(hide yes)
 			(effects
 				(font
@@
 			)
 		)
-		(property "Value" "22K"
-			(at 2.82 -0.02 0)
+		(property "Value" "33K"
+			(at 3.25 -0.019 0)
 			(layer "F.SilkS")
 			(effects
@@
 			(layers "F.Cu" "F.Mask" "F.Paste")
 			(roundrect_rratio 0.208333)
-			(net "Net-(18V3-A)")
+			(net "Net-(12V3-A)")
 			(pintype "passive")
 		)
@@
 		(descr "SMD Solder Jumper, 1x1.5mm, rounded Pads, 0.3mm gap, open")
 		(tags "solder jumper open")
-		(property "Reference" "18V3"
+		(property "Reference" "12V3"
 			(at 0.055 1.835 0)
 			(layer "F.SilkS")
@@
 			(size 1 0.5)
 			(layers "F.Cu" "F.Mask")
-			(net "Net-(18V3-A)")
+			(net "Net-(12V3-A)")
 			(pinfunction "A_1")
 			(pintype "passive")
@@
 			)
 		)
-		(property "Value" "HCR"
+		(property "Value" "Hcr"
 			(at 2.51 4.23 90)
 			(layer "F.SilkS")
@@
 	)
 	(segment
-		(start 167.14 120.83)
-		(end 164.45 120.83)
-		(width 0.2)
-		(layer "F.Cu")
-		(net "Net-(12V2-B)")
-	)
-	(segment
-		(start 164.45 120.83)
-		(end 164.415 120.795)
-		(width 0.2)
-		(layer "F.Cu")
-		(net "Net-(12V2-B)")
-	)
-	(segment
 		(start 146.06 96.86)
 		(end 144.74 95.54)
@@
 	)
 	(segment
-		(start 164.44 124.37)
-		(end 164.415 124.345)
-		(width 0.2)
-		(layer "F.Cu")
-		(net "Net-(9V1-A)")
-	)
-	(segment
-		(start 167.1 124.37)
-		(end 164.44 124.37)
-		(width 0.2)
-		(layer "F.Cu")
-		(net "Net-(9V1-A)")
-	)
-	(segment
 		(start 134.27 110.94)
 		(end 134.95 110.94)
@@
 	)
 	(segment
-		(start 167.2 117.24)
-		(end 164.42 117.24)
-		(width 0.2)
-		(layer "F.Cu")
-		(net "Net-(18V3-A)")
-	)
-	(segment
-		(start 164.42 117.24)
-		(end 164.415 117.245)
-		(width 0.2)
-		(layer "F.Cu")
-		(net "Net-(18V3-A)")
-	)
-	(segment
 		(start 159.08 97.47)
 		(end 159.625 96.925)
@@
 		(net "Net-(U6-VCC)")
 	)
+	(segment
+		(start 164.44 124.37)
+		(end 164.415 124.345)
+		(width 0.2)
+		(layer "F.Cu")
+		(net "Net-(6V1-A)")
+	)
+	(segment
+		(start 167.1 124.37)
+		(end 164.44 124.37)
+		(width 0.2)
+		(layer "F.Cu")
+		(net "Net-(6V1-A)")
+	)
+	(segment
+		(start 167.14 120.83)
+		(end 164.45 120.83)
+		(width 0.2)
+		(layer "F.Cu")
+		(net "Net-(9V2-B)")
+	)
+	(segment
+		(start 164.45 120.83)
+		(end 164.415 120.795)
+		(width 0.2)
+		(layer "F.Cu")
+		(net "Net-(9V2-B)")
+	)
+	(segment
+		(start 167.2 117.24)
+		(end 164.42 117.24)
+		(width 0.2)
+		(layer "F.Cu")
+		(net "Net-(12V3-A)")
+	)
+	(segment
+		(start 164.42 117.24)
+		(end 164.415 117.245)
+		(width 0.2)
+		(layer "F.Cu")
+		(net "Net-(12V3-A)")
+	)
 	(zone

Commit message: Add files via upload
Parts:
- Q1: value AOD4184 -> AOD4185
Changed lines of the file:
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@@
 			)
 		)
-		(property "Value" "AOD4184"
+		(property "Value" "AOD4185"
 			(at 0 4.5 0)
 			(layer "F.SilkS")
@@
 	)
 	(segment
+		(start 167.14 120.83)
+		(end 164.45 120.83)
+		(width 0.2)
+		(layer "F.Cu")
+		(net "Net-(9V2-B)")
+	)
+	(segment
+		(start 164.45 120.83)
+		(end 164.415 120.795)
+		(width 0.2)
+		(layer "F.Cu")
+		(net "Net-(9V2-B)")
+	)
+	(segment
 		(start 146.06 96.86)
 		(end 144.74 95.54)
@@
 	)
 	(segment
+		(start 164.44 124.37)
+		(end 164.415 124.345)
+		(width 0.2)
+		(layer "F.Cu")
+		(net "Net-(6V1-A)")
+	)
+	(segment
+		(start 167.1 124.37)
+		(end 164.44 124.37)
+		(width 0.2)
+		(layer "F.Cu")
+		(net "Net-(6V1-A)")
+	)
+	(segment
 		(start 134.27 110.94)
 		(end 134.95 110.94)
@@
 	)
 	(segment
+		(start 167.2 117.24)
+		(end 164.42 117.24)
+		(width 0.2)
+		(layer "F.Cu")
+		(net "Net-(12V3-A)")
+	)
+	(segment
+		(start 164.42 117.24)
+		(end 164.415 117.245)
+		(width 0.2)
+		(layer "F.Cu")
+		(net "Net-(12V3-A)")
+	)
+	(segment
 		(start 159.08 97.47)
 		(end 159.625 96.925)
@@
 		(net "Net-(U6-VCC)")
 	)
-	(segment
-		(start 164.44 124.37)
-		(end 164.415 124.345)
-		(width 0.2)
-		(layer "F.Cu")
-		(net "Net-(6V1-A)")
-	)
-	(segment
-		(start 167.1 124.37)
-		(end 164.44 124.37)
-		(width 0.2)
-		(layer "F.Cu")
-		(net "Net-(6V1-A)")
-	)
-	(segment
-		(start 167.14 120.83)
-		(end 164.45 120.83)
-		(width 0.2)
-		(layer "F.Cu")
-		(net "Net-(9V2-B)")
-	)
-	(segment
-		(start 164.45 120.83)
-		(end 164.415 120.795)
-		(width 0.2)
-		(layer "F.Cu")
-		(net "Net-(9V2-B)")
-	)
-	(segment
-		(start 167.2 117.24)
-		(end 164.42 117.24)
-		(width 0.2)
-		(layer "F.Cu")
-		(net "Net-(12V3-A)")
-	)
-	(segment
-		(start 164.42 117.24)
-		(end 164.415 117.245)
-		(width 0.2)
-		(layer "F.Cu")
-		(net "Net-(12V3-A)")
-	)
 	(zone
