File: hardware/Water-level-esp8266-esphome-solar-charing.kicad_sch (KiCad schematic)
At the start: 64 parts, among them J1 RESET, J2 FLASH, J3 TTL, J4 Hcr, J5 BATTERY, J6 SOLAR PANEL, Q1 AOD4184, Q2 FS8205A, U1 ESP-12E, U2 AMS1117-3.3, U3 MT3608, U4 INA219AxD, U5 CN3791, U6 DW01A

Commit message: Add files via upload
Parts:
- removed R17: 56K, Resistor_SMD:R_0805_2012Metric_Pad1.20x1.40mm_HandSolder, symbol Device:R
- R13: value 100K -> 68K
- R14: value 43K -> 39K
- R15: value 22K -> 33K
- renumbered 18V3 to 12V3, 9V1 to 6V1, 12V2 to 9V2
Changed lines of the file:
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@@
 	)
 	(junction
-		(at 60.452 160.02)
-		(diameter 0)
-		(color 0 0 0 0)
-	)
-	(junction
 		(at 44.704 129.54)
 		(diameter 0)
@@
 	)
 	(junction
-		(at 70.612 184.912)
-		(diameter 0)
-		(color 0 0 0 0)
-	)
-	(junction
 		(at 215.9 75.184)
 		(diameter 0)
@@
 	(wire
 		(pts
-			(xy 60.452 170.18) (xy 60.452 160.02)
-		)
-		(stroke
-			(width 0)
-			(type default)
-		)
-	)
-	(wire
-		(pts
 			(xy 156.972 121.92) (xy 156.972 123.952)
 		)
@@
 	(wire
 		(pts
-			(xy 50.546 160.02) (xy 60.452 160.02)
+			(xy 50.546 160.02) (xy 76.454 160.02)
 		)
 		(stroke
@@
 	(wire
 		(pts
-			(xy 60.452 160.02) (xy 76.454 160.02)
-		)
-		(stroke
-			(width 0)
-			(type default)
-		)
-	)
-	(wire
-		(pts
 			(xy 236.22 29.464) (xy 240.03 29.464)
 		)
@@
 	(wire
 		(pts
-			(xy 60.452 184.912) (xy 70.612 184.912)
-		)
-		(stroke
-			(width 0)
-			(type default)
-		)
-	)
-	(wire
-		(pts
 			(xy 220.98 82.804) (xy 215.9 82.804)
 		)
@@
 	(wire
 		(pts
-			(xy 60.452 177.8) (xy 60.452 184.912)
-		)
-		(stroke
-			(width 0)
-			(type default)
-		)
-	)
-	(wire
-		(pts
 			(xy 121.666 52.832) (xy 121.666 56.642)
 		)
@@
 			)
 		)
-		(property "Value" "22K"
+		(property "Value" "33K"
 			(at 76.708 182.88 0)
 			(show_name no)
@@
 		(in_pos_files yes)
 		(dnp no)
-		(property "Reference" "12V2"
+		(property "Reference" "9V2"
 			(at 72.39 165.608 90)
 			(show_name no)
@@
 			(project "Water-level-esp8266-esphome-solar-charing"
 				(path "/c778f974-67ff-4a87-97d2-83ab16b1ed92"
-					(reference "12V2")
+					(reference "9V2")
 					(unit 1)
 				)
@@
 			)
 		)
-		(property "Value" "43K"
+		(property "Value" "39K"
 			(at 72.136 182.88 0)
 			(show_name no)
@@
 		(in_pos_files yes)
 		(dnp no)
-		(property "Reference" "18V3"
+		(property "Reference" "12V3"
 			(at 79.248 165.862 90)
 			(show_name no)
@@
 			(project "Water-level-esp8266-esphome-solar-charing"
 				(path "/c778f974-67ff-4a87-97d2-83ab16b1ed92"
-					(reference "18V3")
+					(reference "12V3")
 					(unit 1)
 				)
@@
 		(in_pos_files yes)
 		(dnp no)
-		(property "Reference" "9V1"
+		(property "Reference" "6V1"
 			(at 67.31 165.608 90)
 			(show_name no)
@@
 			(project "Water-level-esp8266-esphome-solar-charing"
 				(path "/c778f974-67ff-4a87-97d2-83ab16b1ed92"
-					(reference "9V1")
+					(reference "6V1")
 					(unit 1)
 				)
@@
 	)
 	(symbol
-		(lib_id "Device:R")
-		(at 60.452 173.99 0)
-		(unit 1)
-		(body_style 1)
-		(exclude_from_sim no)
-		(in_bom yes)
-		(on_board yes)
-		(in_pos_files yes)
-		(dnp no)
-		(property "Reference" "R17"
-			(at 61.976 172.72 0)
-			(show_name no)
-			(do_not_autoplace no)
-			(effects
-				(font
-					(size 1.27 1.27)
-				)
-				(justify left)
-			)
-		)
-		(property "Value" "56K"
-			(at 61.976 175.26 0)
-			(show_name no)
-			(do_not_autoplace no)
-			(effects
-				(font
-					(size 1.27 1.27)
-				)
-				(justify left)
-			)
-		)
-		(property "Footprint" "Resistor_SMD:R_0805_2012Metric_Pad1.20x1.40mm_HandSolder"
-			(at 58.674 173.99 90)
-			(hide yes)
-			(show_name no)
-			(do_not_autoplace no)
-			(effects
-				(font
-					(size 1.27 1.27)
-				)
-			)
-		)
-		(property "Datasheet" ""
-			(at 60.452 173.99 0)
-			(hide yes)
-			(show_name no)
-			(do_not_autoplace no)
-			(effects
-				(font
-					(size 1.27 1.27)
-				)
-			)
-		)
-		(property "Description" "Resistor"
-			(at 60.452 173.99 0)
-			(hide yes)
-			(show_name no)
-			(do_not_autoplace no)
-			(effects
-				(font
-					(size 1.27 1.27)
-				)
-			)
-		)
-		(property "KiLib_Generator" "SMD_2terminal_chip_molded"
-			(at 60.452 173.99 0)
-			(hide yes)
-			(show_name no)
-			(do_not_autoplace no)
-			(effects
-				(font
-					(size 1.27 1.27)
-				)
-			)
-		)
-		(pin "2"
-		)
-		(pin "1"
-		)
-		(instances
-			(project "Water-level-esp8266-esphome-solar-charing"
-				(path "/c778f974-67ff-4a87-97d2-83ab16b1ed92"
-					(reference "R17")
-					(unit 1)
-				)
-			)
-		)
-	)
-	(symbol
 		(lib_id "Transistor_FET:AO3401A")
 		(at 108.204 124.46 90)
@@
 			)
 		)
-		(property "Value" "100K"
+		(property "Value" "68K"
 			(at 65.786 182.88 0)
 			(show_name no)

Commit message: Add files via upload
Parts:
- Q1: value AOD4184 -> AOD4185
Changed lines of the file:
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@@
 			)
 		)
-		(property "Value" "AOD4184"
+		(property "Value" "AOD4185"
 			(at 108.204 118.11 90)
 			(show_name no)
